Commit message: update the files

File: limo_simulation/urdf/limo_four_diff.xacro (robot description, xacro)
@@ -1,6 +1,6 @@
 <?xml version="1.0"?>
 <robot name="limo_four_diff" xmlns:xacro="http://ros.org/wiki/xacro">
-    <xacro:include filename="$(find limo_description)/urdf/limo_xacro.xacro" />
-    <!-- <xacro:include filename="$(find limo_description)/urdf/limo_four_diff_2.gazebo" /> -->
+    <xacro:include filename="$(find limo_simulation)/urdf/limo_xacro.xacro" />
+    <!-- <xacro:include filename="$(find limo_simulation)/urdf/limo_four_diff_2.gazebo" /> -->
     <!-- Variables -->
     <xacro:property name="M_PI" value="3.14159"/>
@@ -26,5 +26,5 @@
 <!--            <origin xyz="0 0 -0.15" rpy="0 0 1.57" />
             <geometry>
-                <mesh filename="file://$(find limo_description)/meshes/limo_base.dae" scale="1 1 1"/>
+                <mesh filename="file://$(find limo_simulation)/meshes/limo_base.dae" scale="1 1 1"/>
             </geometry>-->
             <origin xyz="0 0 0" rpy="0 0 0" />

File: limo_simulation/urdf/limo_xacro.xacro (robot description, xacro)
@@ -11,5 +11,5 @@
 <!--                <origin xyz="0 0 0" rpy="0 0 0" />
                 <geometry>
-                    <mesh filename="file://$(find limo_description)/meshes/limo_wheel.dae" />
+                    <mesh filename="file://$(find limo_simulation)/meshes/limo_wheel.dae" />
                 </geometry>-->
               <origin xyz="0 ${wheel_length/2} 0" rpy="1.57 0 0" />

Commit message: working on the arena

File: limo_simulation/urdf/limo_four_diff.xacro (robot description, xacro)
@@ -12,5 +12,5 @@
     <xacro:property name="track" value="0.13"/>
     <xacro:property name="wheel_vertical_offset" value="-0.10" />
-    <xacro:property name="base_mass" value="2.1557"/>
+    <xacro:property name="base_mass" value="4.8"/>
     <xacro:property name="wheel_length" value="0.045" />
     <xacro:property name="wheel_radius" value="0.045" />
@@ -37,5 +37,6 @@
             <origin xyz="0 0 0" rpy="0 0 0" />
           <geometry>
-              <box size="${base_x_size} ${base_y_size} ${base_z_size}"/>
+              <!--<box size="${base_x_size} ${base_y_size} ${base_z_size}"/>-->
+            <box size="0.322 0.22 0.251"/>
           </geometry>
         </collision>
@@ -45,7 +46,7 @@
             <origin xyz="0.0 0.0 0.0" />
             <mass value="${base_mass}" />
-            <inertia ixx="0.24" ixy="0" ixz="0"
-                     iyy="0.96" iyz="0"
-                     izz="0.96" />
+            <inertia ixx="0.44" ixy="0" ixz="0"
+                     iyy="0.66" iyz="0"
+                     izz="0.6" />
         </inertial>
     </link>
@@ -244,5 +245,5 @@
         <wheel_separation>0.172</wheel_separation>
         <wheel_diameter>0.09</wheel_diameter>
-        <max_wheel_torque>20</max_wheel_torque>
+        <max_wheel_torque>10</max_wheel_torque>
         <max_wheel_acceleration>1.0</max_wheel_acceleration>
         <command_topic>cmd_vel</command_topic>

File: limo_simulation/urdf/limo_xacro.xacro (robot description, xacro)
@@ -23,4 +23,18 @@
                   <cylinder length="${wheel_length}" radius="${wheel_radius}" />
               </geometry>
+            <surface>
+            <friction>
+                <ode>
+                <mu>1.0</mu>
+                <mu2>1.0</mu2>
+                </ode>
+            </friction>
+            <contact>
+                <ode>
+                <max_vel>0.1</max_vel>
+                <min_depth>0.001</min_depth>
+                </ode>
+            </contact>
+            </surface>
             </collision>
         </link>
